File: crystal.kicad_sch (KiCad schematic)
At the start: 4 parts, among them Y1 Crystal_GND23

Commit message: adding labels and updating PCB
Connections:
- net XIN: now reaches C4.1, Y1.1
- net XOUT: now reaches R2.1
Changed lines of the file:
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@@
+		)
+	)
+	(label "XOUT"
+		(at 176.53 93.98 180)
+		(effects
+			(font
+				(size 1.27 1.27)
+			)
+			(justify right bottom)
+		)
+	)
+	(label "XIN"
+		(at 176.53 80.01 180)
+		(effects
+			(font
+				(size 1.27 1.27)
+			)
+			(justify right bottom)
 		)
 	)
