File: usbpower.kicad_sch (KiCad schematic)
At the start: 4 parts, among them J1 USB_C_Receptacle_USB2.0_14P, U2 NCP1117-3.3_SOT223

Commit message: added oscillator and memory
Parts:
- J1: footprint (none) -> Connector_USB:USB_C_Receptacle_Amphenol_12401610E4-2A
Changed lines of the file:
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@@
 			)
 		)
-		(property "Footprint" ""
+		(property "Footprint" "Connector_USB:USB_C_Receptacle_Amphenol_12401610E4-2A"
 			(at 35.56 54.61 0)
 			(effects

Commit message: adding labels and updating PCB
Connections:
- net USBD+ renamed USB_D+
- net USBD- renamed USB_D-
Changed lines of the file:
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@@
 	(wire
 		(pts
-			(xy 46.99 57.15) (xy 49.53 57.15)
+			(xy 46.99 57.15) (xy 54.61 57.15)
 		)
 		(stroke
@@
 	(wire
 		(pts
-			(xy 46.99 52.07) (xy 49.53 52.07)
+			(xy 46.99 52.07) (xy 54.61 52.07)
 		)
 		(stroke
@@
 		)
 	)
-	(hierarchical_label "USBD+"
-		(shape output)
-		(at 49.53 57.15 0)
+	(label "USB_D+"
+		(at 54.61 57.15 180)
 		(effects
 			(font
 				(size 1.27 1.27)
 			)
-			(justify left)
+			(justify right bottom)
 		)
 	)
-	(hierarchical_label "USBD-"
-		(shape output)
-		(at 49.53 52.07 0)
+	(label "USB_D-"
+		(at 54.61 52.07 180)
 		(effects
 			(font
 				(size 1.27 1.27)
 			)
-			(justify left)
+			(justify right bottom)
 		)
 	)
